File: Section A - Title A.kicad_sch (KiCad schematic)
At the start: 0 parts

Commit message: first attempt
Parts:
- added C401: C, symbol Device:C
- added U401: ESP32-C3-DevKitM-1, RF_Module:ESP32-C3-DevKitM-1, symbol RF_Module:ESP32-C3-DevKitM-1
Connections:
- new net: C401.1, U401.2 (3V3), U401.3 (3V3)
- new net: C401.2, U401.20 (IO4)
- new net: U401.1 (GND), U401.12 (GND), U401.15 (GND), U401.16 (GND), U401.19 (GND), U401.24 (GND), U401.27 (GND), U401.30 (GND), U401.6 (GND), U401.8 (GND)
- new net: U401.13 (5V), U401.14 (5V)
- no-connect marks 0 -> 17
