File: Section A - Title A.kicad_sch (KiCad schematic)
At the start: 2 parts, among them U401 ESP32-C3-DevKitM-1

Commit message: footprint added
Parts:
- C401: footprint (none) -> Capacitor_SMD:C_0805_2012Metric_Pad1.18x1.45mm_HandSolder
Changed lines of the file:
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@@
 			)
 		)
-		(property "Footprint" ""
+		(property "Footprint" "Capacitor_SMD:C_0805_2012Metric_Pad1.18x1.45mm_HandSolder"
 			(at 174.9552 72.39 0)
 			(effects
