File: Section B - TItle B.kicad_sch (KiCad schematic)
At the start: 0 parts

Commit message: second update
Parts:
- added C501: C, symbol Device:C
- added D501: LED, symbol Device:LED
- added R501: R, symbol Device:R
Connections:
- new net: C501.1, D501.1 (K)
- new net: D501.2 (A), R501.2
- new net: C501.2, R501.1
