File: KiBot.kicad_pcb (KiCad board)
At the start: 6 copper layers, 0 parts

Commit message: [Preliminary] Pcb layout added
Parts:
- added C401: C, Capacitor_SMD:C_0805_2012Metric_Pad1.18x1.45mm_HandSolder, F.Cu at (141.2, 74.2)
- added C501: C, Capacitor_SMD:C_0805_2012Metric_Pad1.18x1.45mm_HandSolder, F.Cu at (137.9, 80.8)
- added D501: LED, LED_SMD:LED_0805_2012Metric_Pad1.15x1.40mm_HandSolder, F.Cu at (141.4, 79.6)
- added R501: R, Resistor_SMD:R_0805_2012Metric_Pad1.20x1.40mm_HandSolder, F.Cu at (141.3, 82.6)
- added U401: ESP32-C3-DevKitM-1, RF_Module:ESP32-C3-DevKitM-1, F.Cu at (145.1, 67.6)
Routing:
- net Net-(U401-IO4): track 0.00 -> 34.2 mm
- net Net-(C401-Pad1): track 0.00 -> 4.12 mm
- net Net-(D501-A): track 0.00 -> 3.02 mm
- net Net-(C501-Pad2): track 0.00 -> 2.74 mm
- net Net-(D501-K): track 0.00 -> 2.48 mm
Other:
- board outline added: 39.4 x 48 mm
