File: KiBot.kicad_pcb (KiCad board)
At the start: 6 copper layers, 39.4 x 48 mm, 5 parts, among them U401 ESP32-C3-DevKitM-1

Commit message: [CHECKED] Last check complated
Parts:
- added G***: LOGO, LOGO, F.Cu at (157.4, 84.0)
- C501, D501, R501: moved to B.Cu
- moved C501 21.6 mm to (159.3, 84.2)
- moved R501 14.9 mm to (155.9, 86.0), turned to 180 degrees
- moved D501 14.9 mm to (155.8, 83.0), turned to 180 degrees

Commit message: bugs fixed
Routing:
- net Net-(U401-IO4): track 34.2 -> 40.3 mm
Changed lines of the file:
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@@
 	(property "DESIGNER" "Fate")
 	(property "FABRICATION_NOTES" "FABRICATION NOTES (UNLESS OTHERWISE SPECIFIED)\n\n1)	FABRICATE PER IPC-6012A CLASS 2.\n\n2)	OUTLINE DEFINED IN SEPARATE GERBER FILE WITH\n	\"Edge_Cuts.GBR\" SUFFIX.\n\n	DIMENSIONS OF CIRCUMSIZED RECTANGLE SHOWN ON THIS\n	DRAWING FOR REFERENCE ONLY.\n\n3)	SEE SEPARATE DRILL FILES WITH \".DRL\" SUFFIX \n	FOR HOLE LOCATIONS.\n\n	SELECTED HOLE LOCATIONS SHOWN ON THIS DRAWING \n	FOR REFERENCE ONLY.\n\n4)	SURFACE FINISH: IMMERSION GOLD\n\n5)	SOLDERMASK ON BOTH SIDES OF THE BOARD SHALL \n	BE LPI, COLOR BLACK.\n\n6)	SILK SCREEN LEGEND TO BE APPLIED PER LAYER \n	STACKUP USING YELLOW NON-CONDUCTIVE EPOXY INK.\n\n7)	ALL VIAS ARE TENTED ON BOTH SIDES UNLESS \n	SOLDERMASK OPENED IN GERBER.\n\n8)	VENDOR SHOULD FOLLOW ROHS COMPLIANT PROCESS \n	AND Pb FREE FOR MANUFACTURING\n\n9)	PCB MATERIAL REQUIREMENTS:\n\n	A.	FLAMMABILITY RATING MUST MEET OR EXCEED \n		UL94V-0 REQUIREMENTS.\n	B.	Tg 170 C OR EQUIVALENT.\n	C.	EQUIVALENT MATERIAL SHALL BE RoHS COMPLIANT, \n		HALOGEN FREE AND APPROVED BY SEMRUK.\n\n10)	DESIGN GEOMETRY MINIMUM FEATURE SIZES:\n\n	BOARD SIZE				39.400 × 48.000 mm\n	BOARD THICKNESS		1.660 mm\n	TRACE WIDTH			0.200 mm\n	TRACE TO TRACE		0.200 mm\n	MIN. HOLE (PTH)			0.900 mm\n	MIN. HOLE (NPTH)		N/A mm\n	ANNULAR RING			0.300 mm\n	COPPER TO HOLE		0.254 mm\n	COPPER TO EDGE		0.250 mm\n	HOLE TO HOLE			0.254 mm\n\n11)	REFER TO IMPEDANCE TABLE FOR IMPEDANCE CONTROL REQUIREMENTS.\n\n12)	CONFIRM SPACE WIDTHS AND SPACINGS.")
-	(property "GIT_HASH_PCB" "2259e50")
+	(property "GIT_HASH_PCB" "0e9df05")
 	(property "GIT_HASH_SCH" "68a27aa")
 	(property "GIT_URL" "https://github.com/nguyen-v/KDT_Hierarchical_KiBot")
 	(property "PROJECT_NAME" "KiBot")
-	(property "RELEASE_BODY_1.0.0" "")
+	(property "RELEASE_BODY_1.0.0" "Version 1.0.0 not found.")
 	(property "RELEASE_BODY_1.0.1" "")
 	(property "RELEASE_BODY_1.0.2" "")
@@
 	(property "RELEASE_DATE" "18-Mar-2026")
 	(property "RELEASE_DATE_NUM" "2026-03-18")
-	(property "RELEASE_TITLE_1.0.0" "")
+	(property "RELEASE_TITLE_1.0.0" "Version 1.0.0 not found.")
 	(property "RELEASE_TITLE_1.0.1" "")
 	(property "RELEASE_TITLE_1.0.2" "")
@@
 	(property "SHEET_NAME_8" "......................................")
 	(property "SHEET_NAME_9" "......................................")
-	(property "VARIANT" "PRELIMINARY")
+	(property "VARIANT" "CHECKED")
 	(net 0 "")
 	(net 1 "Net-(C401-Pad1)")
@@
 	)
 	(segment
-		(start 142.7125 76.75)
-		(end 151.71 76.75)
+		(start 146.25 76.4)
+		(end 142.325 76.4)
 		(width 0.2)
 		(layer "F.Cu")
@@
 	)
 	(segment
-		(start 151.71 76.75)
-		(end 168 93.04)
+		(start 150.4 88.84)
+		(end 150.4 80.55)
+		(width 0.2)
+		(layer "F.Cu")
+		(net 2)
+	)
+	(segment
+		(start 142.325 76.4)
+		(end 141.9625 76.0375)
+		(width 0.2)
+		(layer "F.Cu")
+		(net 2)
+	)
+	(segment
+		(start 154.6 93.04)
+		(end 150.4 88.84)
+		(width 0.2)
+		(layer "F.Cu")
+		(net 2)
+	)
+	(segment
+		(start 168 93.04)
+		(end 154.6 93.04)
+		(width 0.2)
+		(layer "F.Cu")
+		(net 2)
+	)
+	(segment
+		(start 147.525 77.675)
+		(end 146.6 76.75)
+		(width 0.2)
+		(layer "F.Cu")
+		(net 2)
+	)
+	(segment
+		(start 150.4 80.55)
+		(end 147.525 77.675)
 		(width 0.2)
 		(layer "F.Cu")
@@
 	(segment
 		(start 141.2 75.275)
-		(end 142.7125 76.7875)
+		(end 141.9625 76.0375)
+		(width 0.2)
+		(layer "F.Cu")
+		(net 2)
+	)
+	(segment
+		(start 147.525 77.675)
+		(end 146.25 76.4)
 		(width 0.2)
 		(layer "F.Cu")

Commit message: bugs fixed v2
Parts:
- moved C401 11.4 mm to (152.6, 75.2)
Routing:
- net Net-(U401-IO4): track 40.3 -> 33.1 mm
- net Net-(C401-Pad1): track 4.12 -> 11.2 mm
Other:
- board size 39.4 x 48 mm -> 25.6 x 41.8 mm
Changed lines of the file:
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@@
 	(property "DESIGNER" "Fate")
 	(property "FABRICATION_NOTES" "FABRICATION NOTES (UNLESS OTHERWISE SPECIFIED)\n\n1)	FABRICATE PER IPC-6012A CLASS 2.\n\n2)	OUTLINE DEFINED IN SEPARATE GERBER FILE WITH\n	\"Edge_Cuts.GBR\" SUFFIX.\n\n	DIMENSIONS OF CIRCUMSIZED RECTANGLE SHOWN ON THIS\n	DRAWING FOR REFERENCE ONLY.\n\n3)	SEE SEPARATE DRILL FILES WITH \".DRL\" SUFFIX \n	FOR HOLE LOCATIONS.\n\n	SELECTED HOLE LOCATIONS SHOWN ON THIS DRAWING \n	FOR REFERENCE ONLY.\n\n4)	SURFACE FINISH: IMMERSION GOLD\n\n5)	SOLDERMASK ON BOTH SIDES OF THE BOARD SHALL \n	BE LPI, COLOR BLACK.\n\n6)	SILK SCREEN LEGEND TO BE APPLIED PER LAYER \n	STACKUP USING YELLOW NON-CONDUCTIVE EPOXY INK.\n\n7)	ALL VIAS ARE TENTED ON BOTH SIDES UNLESS \n	SOLDERMASK OPENED IN GERBER.\n\n8)	VENDOR SHOULD FOLLOW ROHS COMPLIANT PROCESS \n	AND Pb FREE FOR MANUFACTURING\n\n9)	PCB MATERIAL REQUIREMENTS:\n\n	A.	FLAMMABILITY RATING MUST MEET OR EXCEED \n		UL94V-0 REQUIREMENTS.\n	B.	Tg 170 C OR EQUIVALENT.\n	C.	EQUIVALENT MATERIAL SHALL BE RoHS COMPLIANT, \n		HALOGEN FREE AND APPROVED BY SEMRUK.\n\n10)	DESIGN GEOMETRY MINIMUM FEATURE SIZES:\n\n	BOARD SIZE				39.400 × 48.000 mm\n	BOARD THICKNESS		1.660 mm\n	TRACE WIDTH			0.200 mm\n	TRACE TO TRACE		0.200 mm\n	MIN. HOLE (PTH)			0.900 mm\n	MIN. HOLE (NPTH)		N/A mm\n	ANNULAR RING			0.300 mm\n	COPPER TO HOLE		0.254 mm\n	COPPER TO EDGE		0.250 mm\n	HOLE TO HOLE			0.254 mm\n\n11)	REFER TO IMPEDANCE TABLE FOR IMPEDANCE CONTROL REQUIREMENTS.\n\n12)	CONFIRM SPACE WIDTHS AND SPACINGS.")
-	(property "GIT_HASH_PCB" "0e9df05")
+	(property "GIT_HASH_PCB" "32e13b4")
 	(property "GIT_HASH_SCH" "68a27aa")
 	(property "GIT_URL" "https://github.com/nguyen-v/KDT_Hierarchical_KiBot")
@@
 	(footprint "Capacitor_SMD:C_0805_2012Metric_Pad1.18x1.45mm_HandSolder"
 		(layer "F.Cu")
-		(at 141.2 74.2375 -90)
+		(at 152.6 75.2 -90)
 		(descr "Capacitor SMD 0805 (2012 Metric), square (rectangular) end terminal, IPC_7351 nominal with elongated pad for handsoldering. (Body size source: IPC-SM-782 page 76, https://www.pcb-3d.com/wordpress/wp-content/uploads/ipc-sm-782a_amendment_1_and_2.pdf, https://docs.google.com/spreadsheets/d/1BsfQQcO9C6DZCsRaXUlFlo91Tg2WpOkGARC1WS5S8t0/edit?usp=sharing), generated with kicad-footprint-generator")
 		(tags "capacitor handsolder")
@@
 	)
 	(gr_line
-		(start 173.2 59.6)
-		(end 173.2 107.6)
+		(start 169.4 65.8)
+		(end 169.4 107.6)
 		(stroke
 			(width 0.1)
@@
 	)
 	(gr_line
-		(start 173.2 107.6)
-		(end 133.8 107.6)
+		(start 169.4 107.6)
+		(end 143.8 107.6)
 		(stroke
 			(width 0.1)
@@
 	)
 	(gr_line
-		(start 133.8 59.6)
-		(end 173.2 59.6)
+		(start 143.8 65.8)
+		(end 169.4 65.8)
 		(stroke
 			(width 0.1)
@@
 	)
 	(gr_line
-		(start 133.8 107.6)
-		(end 133.8 59.6)
+		(start 143.8 107.6)
+		(end 143.8 65.8)
 		(stroke
 			(width 0.1)
@@
 	)
 	(segment
-		(start 141.2 73.2)
-		(end 144.6975 73.2)
+		(start 151.1575 72.72)
+		(end 152.6 74.1625)
 		(width 0.2)
 		(layer "F.Cu")
@@
 	)
 	(segment
-		(start 146.25 76.4)
-		(end 142.325 76.4)
+		(start 145.14 72.72)
+		(end 151.1575 72.72)
 		(width 0.2)
 		(layer "F.Cu")
-		(net 2)
+		(net 1)
 	)
 	(segment
-		(start 150.4 88.84)
-		(end 150.4 80.55)
+		(start 145.14 70.18)
+		(end 145.14 72.72)
 		(width 0.2)
 		(layer "F.Cu")
-		(net 2)
+		(net 1)
 	)
 	(segment
-		(start 142.325 76.4)
-		(end 141.9625 76.0375)
+		(start 152.6 78.4)
+		(end 152.6 76.2375)
 		(width 0.2)
 		(layer "F.Cu")
@@
 	)
 	(segment
-		(start 168 93.04)
-		(end 154.6 93.04)
+		(start 150.4 80.8)
+		(end 150.4 80.6)
 		(width 0.2)
 		(layer "F.Cu")
@@
 	)
 	(segment
-		(start 147.525 77.675)
-		(end 146.6 76.75)
+		(start 168 93.04)
+		(end 154.6 93.04)
 		(width 0.2)
 		(layer "F.Cu")
@@
 	)
 	(segment
-		(start 150.4 80.55)
-		(end 147.525 77.675)
+		(start 150.4 88.84)
+		(end 150.4 80.8)
 		(width 0.2)
 		(layer "F.Cu")
@@
 	)
 	(segment
-		(start 141.2 75.275)
-		(end 141.9625 76.0375)
+		(start 150.4 80.8)
+		(end 150.4 80.55)
 		(width 0.2)
 		(layer "F.Cu")
@@
 	)
 	(segment
-		(start 147.525 77.675)
-		(end 146.25 76.4)
+		(start 150.4 80.6)
+		(end 152.6 78.4)
 		(width 0.2)
 		(layer "F.Cu")

Commit message: bugs fixed v3
Routing:
- net Net-(C401-Pad1): track 11.2 -> 20.9 mm
